Commit message: Testing Libserial

File: description/urdf/levibot.core.xacro (robot description, xacro)
@@ -136,3 +136,26 @@
     </xacro:inertial_cylinder>
   </link>
+  <!-- Sensors -->
+  <!-- IMU Link -->
+  <joint name="imu_joint" type="fixed">
+    <origin xyz="0.0 0.0 0.03" rpy="0.0 0.0 0.0"/>
+    <parent link="base_link"/>
+    <child link="imu_link"/>
+  </joint>
+  <link name="imu_link">
+    <collision>
+      <geometry>
+        <box size="0.025 0.02 0.005"/>
+      </geometry>
+    </collision>
+    <visual>
+      <geometry>
+        <box size="0.025 0.02 0.005"/>
+      </geometry>
+      <material name="white" />
+    </visual>
+    <xacro:inertial_box mass="0.005" x="0.025" y="0.02" z="0.005">
+      <origin xyz="0 0 0" rpy="0 0 0"/>
+    </xacro:inertial_box>
+  </link>
 </robot>

File: description/urdf/levibot.gazebo.xacro (robot description, xacro)
@@ -5,54 +5,40 @@
   </gazebo>
   <gazebo reference="rl_wheel_link">
-    <mu1>0.7</mu1>
-    <mu2>0.7</mu2>
-    <kp>500000.0</kp>
-    <kd>10.0</kd>
-    <minDepth>0.001</minDepth>
-    <maxVel>0.1</maxVel>
-    <fdir1>1 0 0</fdir1>
+    <mu1>0.2</mu1>
+    <mu2>0.2</mu2>
     <material>Gazebo/Grey</material>
   </gazebo>
   <gazebo reference="rr_wheel_link">
-    <mu1>0.7</mu1>
-    <mu2>0.7</mu2>
-    <kp>500000.0</kp>
-    <kd>10.0</kd>
-    <minDepth>0.001</minDepth>
-    <maxVel>0.1</maxVel>
-    <fdir1>1 0 0</fdir1>
+    <mu1>0.2</mu1>
+    <mu2>0.2</mu2>
     <material>Gazebo/Grey</material>
   </gazebo>
   <gazebo reference="fr_wheel_link">
-    <mu1>0.7</mu1>
-    <mu2>0.7</mu2>
-    <kp>500000.0</kp>
-    <kd>10.0</kd>
-    <minDepth>0.001</minDepth>
-    <maxVel>0.1</maxVel>
-    <fdir1>1 0 0</fdir1>
+    <mu1>0.2</mu1>
+    <mu2>0.2</mu2>
     <material>Gazebo/Grey</material>
   </gazebo>
   <gazebo reference="fl_wheel_link">
-    <mu1>0.7</mu1>
-    <mu2>0.7</mu2>
-    <kp>500000.0</kp>
-    <kd>10.0</kd>
-    <minDepth>0.001</minDepth>
-    <maxVel>0.1</maxVel>
-    <fdir1>1 0 0</fdir1>
+    <mu1>0.2</mu1>
+    <mu2>0.2</mu2>
     <material>Gazebo/Grey</material>
   </gazebo>
-<gazebo reference="fl_wheel_hinge">
-       <implicitSpringDamper>true</implicitSpringDamper>
-</gazebo>
-<gazebo reference="fr_wheel_hinge">
-       <implicitSpringDamper>true</implicitSpringDamper>
-</gazebo>
-<gazebo reference="rr_wheel_hinge">
-       <implicitSpringDamper>true</implicitSpringDamper>
-</gazebo>
-<gazebo reference="rl_wheel_hinge">
-       <implicitSpringDamper>true</implicitSpringDamper>
-</gazebo>
+  <gazebo reference="imu_link">
+    <gravity>true</gravity>
+    <material>Gazebo/Grey</material>
+    <sensor name="imu_sensor" type="imu">
+      <always_on>true</always_on>
+      <plugin filename="libgazebo_ros_imu_sensor.so" name="imu">
+        <bodyName>imu_link</bodyName>
+        <gaussianNoise>0.0</gaussianNoise>
+        <xyzOffset>0 0 0</xyzOffset>
+        <rpyOffset>0 0 0</rpyOffset>
+        <frameName>imu_link</frameName>
+        <initialOrientationAsReference>false</initialOrientationAsReference>
+        <ros>
+          <remapping>/imu/out:=/imu</remapping>
+        </ros>
+      </plugin>
+    </sensor>
+  </gazebo>
 </robot>

File: description/urdf/levibot.sim_ros2_control.xacro (robot description, xacro)
@@ -41,5 +41,8 @@
   <gazebo>
     <plugin name="gazebo_ros2_control" filename="libgazebo_ros2_control.so">
-      <parameters>$(find levibot_diffdrive)/config/controllers.yaml</parameters>
+      <parameters>$(find levibot_diffdrive)/config/gz_controllers.yaml</parameters>
+        <ros>
+          <remapping>/base_controller/cmd_vel_unstamped:=/cmd_vel</remapping>
+        </ros>
     </plugin>
   </gazebo>

File: description/urdf/levibot.urdf.xacro (robot description, xacro)
@@ -2,6 +2,6 @@
 <robot xmlns:xacro="http://ros.org/wiki/xacro" name="diffdrive_levibot">
   <xacro:include filename="$(find levibot_diffdrive)/urdf/levibot.core.xacro"/>
-  <xacro:include filename="$(find levibot_diffdrive)/urdf/levibot.ros2_control.xacro"/>
-  <!-- <xacro:include filename="$(find levibot_diffdrive)/urdf/levibot.sim_ros2_control.xacro"/> -->
-  <!-- <xacro:include filename="$(find levibot_diffdrive)/urdf/levibot.gazebo.xacro"/> -->
+  <xacro:include filename="$(find levibot_diffdrive)/urdf/levibot.sim_ros2_control.xacro"/>
+  <xacro:include filename="$(find levibot_diffdrive)/urdf/levibot.gazebo.xacro"/>
+  <!-- <xacro:include filename="$(find levibot_diffdrive)/urdf/levibot.ros2_control.xacro"/> -->
 </robot>

Commit message: Update to ros rolling and gazebo fortress

File: description/urdf/levibot.core.xacro (robot description, xacro)
@@ -2,14 +2,7 @@
 <robot xmlns:xacro="http://ros.org/wiki/xacro">
   <!-- ============= Materials & Intertias =============  -->
-  <xacro:include filename="$(find levibot_diffdrive)/urdf/inertial_macros.xacro"/>
-  <xacro:include filename="$(find levibot_diffdrive)/urdf/materials.xacro"/>
+  <xacro:include filename="$(find levibot_skidsteer)/urdf/inertial_macros.xacro"/>
+  <xacro:include filename="$(find levibot_skidsteer)/urdf/materials.xacro"/>
   <!-- =============== Links & Joints =============== -->
-  <link name="base_footprint"/>
-  <!-- Base Link -->
-  <joint name="base_link_joint" type="fixed">
-    <origin xyz="0 0 0.045"/>
-    <parent link="base_footprint"/>
-    <child link="base_link"/>
-  </joint>
   <link name="base_link"/>
   <!-- Chassis Link  -->

File: description/urdf/levibot.gazebo.xacro (robot description, xacro)
@@ -42,3 +42,34 @@
     </sensor>
   </gazebo>
+  <gazebo>
+    <plugin name='skid_steer_drive' filename='libgazebo_ros_diff_drive.so'>
+      <!-- <ros>
+        <namespace>/demo</namespace>
+        <argument>cmd_vel:=cmd_demo</argument>
+        <argument>odom:=odom_demo</argument>
+      </ros> -->
+      <!-- Number of wheel pairs -->
+      <num_wheel_pairs>2</num_wheel_pairs>
+      <!-- wheels0 -->
+      <left_joint>fl_wheel_joint</left_joint>
+      <right_joint>fr_wheel_joint</right_joint>
+      <!-- wheels1-->
+      <left_joint>rl_wheel_joint</left_joint>
+      <right_joint>rr_wheel_joint</right_joint>
+      <!-- kinematics -->
+      <wheel_separation>1.25</wheel_separation>
+      <wheel_separation>1.25</wheel_separation>
+      <wheel_diameter>0.06</wheel_diameter>
+      <wheel_diameter>0.06</wheel_diameter>
+      <!-- limits -->
+      <max_wheel_torque>20</max_wheel_torque>
+      <max_wheel_acceleration>1.0</max_wheel_acceleration>
+      <!-- output -->
+      <publish_odom>true</publish_odom>
+      <publish_odom_tf>true</publish_odom_tf>
+      <publish_wheel_tf>true</publish_wheel_tf>
+      <odometry_frame>odom</odometry_frame>
+      <robot_base_frame>chassis</robot_base_frame>
+    </plugin>
+  </gazebo>
 </robot>

File: description/urdf/levibot.urdf.xacro (robot description, xacro)
@@ -1,7 +1,37 @@
 <?xml version="1.0" encoding="utf-8"?>
 <robot xmlns:xacro="http://ros.org/wiki/xacro" name="diffdrive_levibot">
-  <xacro:include filename="$(find levibot_diffdrive)/urdf/levibot.core.xacro"/>
-  <xacro:include filename="$(find levibot_diffdrive)/urdf/levibot.sim_ros2_control.xacro"/>
-  <xacro:include filename="$(find levibot_diffdrive)/urdf/levibot.gazebo.xacro"/>
-  <!-- <xacro:include filename="$(find levibot_diffdrive)/urdf/levibot.ros2_control.xacro"/> -->
+  <!-- paramters to be set from the launch file -->
+  <xacro:arg name="use_mock_hardware" default="false" />
+  <xacro:arg name="sim_gazebo_classic" default="false" />
+  <xacro:arg name="sim_gazebo" default="false" />
+  <xacro:arg name="simulation_controllers" default="" />
+  <xacro:include filename="$(find levibot_skidsteer)/urdf/levibot.core.xacro"/>
+  <xacro:include filename="$(find levibot_skidsteer)/ros2_control/levibot.ros2_control.xacro"/>
+  <xacro:levibot_ros2_control
+    name="levibot"
+    use_mock_hardware="$(arg use_mock_hardware)"
+    sim_gazebo_classic="$(arg sim_gazebo_classic)"
+    sim_gazebo="$(arg sim_gazebo)"/>
+  <xacro:if value="$(arg sim_gazebo_classic)">
+    <gazebo>
+      <plugin filename="libgazebo_ros2_control.so" name="gazebo_ros2_control">
+        <parameters>$(arg simulation_controllers)</parameters>
+        <ros>
+          <remapping>/base_controller/cmd_vel_unstamped:=/cmd_vel</remapping>
+        </ros>
+      </plugin>
+    </gazebo>
+  </xacro:if>
+  <xacro:if value="$(arg sim_gazebo)">
+    <gazebo>
+        <plugin filename="libgz_ros2_control-system.so" name="gz_ros2_control::GazeboSimROS2ControlPlugin">
+        <parameters>$(arg simulation_controllers)</parameters>
+        <controller_manager_prefix_node_name>controller_manager</controller_manager_prefix_node_name>
+        <ros>
+          <remapping>/base_controller/cmd_vel_unstamped:=/cmd_vel</remapping>
+          <remapping>/base_controller/odom:=/odom</remapping>
+        </ros>
+      </plugin>
+    </gazebo>
+  </xacro:if>
 </robot>

Commit message: Add lidar

File: description/urdf/levibot.core.xacro (robot description, xacro)
@@ -152,3 +152,25 @@
     </xacro:inertial_box>
   </link>
+  <!-- LIDAR Link -->
+  <joint name="lidar_joint" type="fixed">
+    <origin xyz="-0.1 0.0 0.03" rpy="0.0 0.0 0.0"/>
+    <parent link="base_link"/>
+    <child link="lidar_link"/>
+  </joint>
+  <link name="lidar_link">
+    <collision>
+      <geometry>
+        <box size="0.03 0.03 0.025"/>
+      </geometry>
+    </collision>
+    <visual>
+      <geometry>
+        <box size="0.03 0.03 0.025"/>
+      </geometry>
+      <material name="red" />
+    </visual>
+    <xacro:inertial_box mass="0.007" x="0.03" y="0.03" z="0.025">
+      <origin xyz="0 0 0" rpy="0 0 0"/>
+    </xacro:inertial_box>
+  </link>
 </robot>

File: description/urdf/levibot.urdf.xacro (robot description, xacro)
@@ -14,4 +14,5 @@
     sim_gazebo="$(arg sim_gazebo)"/>
   <xacro:if value="$(arg sim_gazebo_classic)">
+    <xacro:include filename="$(find levibot_skidsteer)/urdf/levibot.gazebo.xacro"/>
     <gazebo>
       <plugin filename="libgazebo_ros2_control.so" name="gazebo_ros2_control">
@@ -24,4 +25,5 @@
   </xacro:if>
   <xacro:if value="$(arg sim_gazebo)">
+    <xacro:include filename="$(find levibot_skidsteer)/urdf/levibot.gazebo.xacro"/>
     <gazebo>
         <plugin filename="libgz_ros2_control-system.so" name="gz_ros2_control::GazeboSimROS2ControlPlugin">

File: simulation/urdf/levibot.gazebo.xacro (robot description, xacro)
@@ -42,28 +42,58 @@
     </sensor>
   </gazebo>
-  <gazebo>
+  <gazebo reference="lidar_link">
+    <sensor name='gpu_lidar' type='gpu_lidar'>
+      <pose>0 0 0 0 -0 0</pose>
+      <topic>scan</topic>
+      <update_rate>10</update_rate>
+      <enable_metrics>false</enable_metrics>
+      <lidar>
+        <scan>
+          <horizontal>
+            <samples>640</samples>
+            <resolution>1</resolution>
+            <min_angle>-1.3962600000000001</min_angle>
+            <max_angle>1.3962600000000001</max_angle>
+          </horizontal>
+          <vertical>
+            <samples>16</samples>
+            <min_angle>-0.261799</min_angle>
+            <max_angle>0.261799</max_angle>
+            <resolution>1</resolution>
+          </vertical>
+        </scan>
+        <range>
+          <min>0.080000000000000002</min>
+          <max>10</max>
+          <resolution>0.01</resolution>
+        </range>
+        <noise>
+          <type>none</type>
+          <mean>0</mean>
+          <stddev>0</stddev>
+        </noise>
+        <visibility_mask>4294967295</visibility_mask>
+      </lidar>
+    </sensor>
+  </gazebo>
+  <!-- Using ROS2 Control Instead -->
+  <!-- <gazebo>
     <plugin name='skid_steer_drive' filename='libgazebo_ros_diff_drive.so'>
-      <!-- <ros>
+      <ros>
         <namespace>/demo</namespace>
         <argument>cmd_vel:=cmd_demo</argument>
         <argument>odom:=odom_demo</argument>
-      </ros> -->
-      <!-- Number of wheel pairs -->
+      </ros>
       <num_wheel_pairs>2</num_wheel_pairs>
-      <!-- wheels0 -->
       <left_joint>fl_wheel_joint</left_joint>
       <right_joint>fr_wheel_joint</right_joint>
-      <!-- wheels1-->
       <left_joint>rl_wheel_joint</left_joint>
       <right_joint>rr_wheel_joint</right_joint>
-      <!-- kinematics -->
       <wheel_separation>1.25</wheel_separation>
       <wheel_separation>1.25</wheel_separation>
       <wheel_diameter>0.06</wheel_diameter>
       <wheel_diameter>0.06</wheel_diameter>
-      <!-- limits -->
       <max_wheel_torque>20</max_wheel_torque>
       <max_wheel_acceleration>1.0</max_wheel_acceleration>
-      <!-- output -->
       <publish_odom>true</publish_odom>
       <publish_odom_tf>true</publish_odom_tf>
@@ -72,4 +102,4 @@
       <robot_base_frame>chassis</robot_base_frame>
     </plugin>
-  </gazebo>
+  </gazebo> -->
 </robot>

Commit message: Solved the reverse odom problem with  wheels  z

File: description/urdf/levibot.core.xacro (robot description, xacro)
@@ -34,5 +34,5 @@
     <parent link="base_link"/>
     <child link="fr_wheel_link"/>
-    <axis xyz="0 0 1"/>
+    <axis xyz="0 0 -1"/>
   </joint>
   <link name="fr_wheel_link">
@@ -59,5 +59,5 @@
     <parent link="base_link"/>
     <child link="fl_wheel_link"/>
-    <axis xyz="0 0 -1"/>
+    <axis xyz="0 0 1"/>
   </joint>
   <link name="fl_wheel_link">
@@ -84,5 +84,5 @@
     <parent link="base_link"/>
     <child link="rr_wheel_link"/>
-    <axis xyz="0 0 1"/>
+    <axis xyz="0 0 -1"/>
   </joint>
   <link name="rr_wheel_link">
@@ -109,5 +109,5 @@
     <parent link="base_link"/>
     <child link="rl_wheel_link"/>
-    <axis xyz="0 0 -1"/>
+    <axis xyz="0 0 1"/>
   </joint>
   <link name="rl_wheel_link">
@@ -154,9 +154,9 @@
   <!-- LIDAR Link -->
   <joint name="lidar_joint" type="fixed">
-    <origin xyz="-0.1 0.0 0.03" rpy="0.0 0.0 0.0"/>
+    <origin xyz="0.1 0.0 0.03" rpy="0.0 0.0 0.0"/>
     <parent link="base_link"/>
-    <child link="lidar_link"/>
+    <child link="levibot/base_link/lidar"/>
   </joint>
-  <link name="lidar_link">
+  <link name="levibot/base_link/lidar">
     <collision>
       <geometry>

File: description/urdf/levibot.urdf.xacro (robot description, xacro)
@@ -1,4 +1,4 @@
 <?xml version="1.0" encoding="utf-8"?>
-<robot xmlns:xacro="http://ros.org/wiki/xacro" name="diffdrive_levibot">
+<robot xmlns:xacro="http://ros.org/wiki/xacro" name="levibot">
   <!-- paramters to be set from the launch file -->
   <xacro:arg name="use_mock_hardware" default="false" />

File: simulation/urdf/levibot.gazebo.xacro (robot description, xacro)
@@ -42,10 +42,10 @@
     </sensor>
   </gazebo>
-  <gazebo reference="lidar_link">
-    <sensor name='gpu_lidar' type='gpu_lidar'>
-      <pose>0 0 0 0 -0 0</pose>
+  <gazebo reference="levibot/base_link/lidar">
+    <sensor name='lidar' type='gpu_lidar'>
+      <pose>0 0 0 0 0 0</pose>
       <topic>scan</topic>
-      <update_rate>10</update_rate>
-      <enable_metrics>false</enable_metrics>
+      <update_rate>1000</update_rate>
+      <enable_metrics>true</enable_metrics>
       <lidar>
         <scan>
@@ -53,6 +53,6 @@
             <samples>640</samples>
             <resolution>1</resolution>
-            <min_angle>-1.3962600000000001</min_angle>
-            <max_angle>1.3962600000000001</max_angle>
+            <min_angle>-3.14159</min_angle>
+            <max_angle>3.14159</max_angle>
           </horizontal>
           <vertical>

Commit message: ...

File: description/urdf/levibot.core.xacro (robot description, xacro)
@@ -156,7 +156,7 @@
     <origin xyz="0.1 0.0 0.03" rpy="0.0 0.0 0.0"/>
     <parent link="base_link"/>
-    <child link="levibot/base_link/lidar"/>
+    <child link="lidar_link"/>
   </joint>
-  <link name="levibot/base_link/lidar">
+  <link name="lidar_link">
     <collision>
       <geometry>

File: simulation/urdf/levibot.gazebo.xacro (robot description, xacro)
@@ -2,29 +2,29 @@
 <robot xmlns:xacro="http://ros.org/wiki/xacro">
   <gazebo reference="chassis">
-    <material>Gazebo/White</material>
+    <material>Gazebo/Blue</material>
   </gazebo>
   <gazebo reference="rl_wheel_link">
     <mu1>0.2</mu1>
     <mu2>0.2</mu2>
-    <material>Gazebo/Grey</material>
+    <material>Gazebo/Green</material>
   </gazebo>
   <gazebo reference="rr_wheel_link">
     <mu1>0.2</mu1>
     <mu2>0.2</mu2>
-    <material>Gazebo/Grey</material>
+    <material>Gazebo/Green</material>
   </gazebo>
   <gazebo reference="fr_wheel_link">
     <mu1>0.2</mu1>
     <mu2>0.2</mu2>
-    <material>Gazebo/Grey</material>
+    <material>Gazebo/Green</material>
   </gazebo>
   <gazebo reference="fl_wheel_link">
     <mu1>0.2</mu1>
     <mu2>0.2</mu2>
-    <material>Gazebo/Grey</material>
+    <material>Gazebo/Green</material>
   </gazebo>
   <gazebo reference="imu_link">
     <gravity>true</gravity>
-    <material>Gazebo/Grey</material>
+    <material>Gazebo/Green</material>
     <sensor name="imu_sensor" type="imu">
       <always_on>true</always_on>
@@ -43,6 +43,6 @@
   </gazebo>
   <gazebo reference="levibot/base_link/lidar">
-    <sensor name='lidar' type='gpu_lidar'>
-      <pose relative_to='levibot/base_link/lidar'>0 0 0 0 0 0</pose>
+    <sensor name='levibot_lidar' type='ray'>
+      <pose>0 0 0 0 0 0</pose>
       <topic>scan</topic>
       <update_rate>100</update_rate>
@@ -52,23 +52,36 @@
           <scan>
               <horizontal>
-                  <samples>640</samples>
+                  <samples>720</samples>
                   <resolution>1</resolution>
-                  <min_angle>-1.396263</min_angle>
-                  <max_angle>1.396263</max_angle>
+                  <min_angle>-1.570796</min_angle>
+                  <max_angle>1.570796</max_angle>
               </horizontal>
-              <vertical>
+              <!-- <vertical>
                   <samples>1</samples>
                   <resolution>0.01</resolution>
                   <min_angle>0</min_angle>
                   <max_angle>0</max_angle>
-              </vertical>
+              </vertical> -->
           </scan>
           <range>
               <min>0.08</min>
-              <max>10.0</max>
+              <max>20.0</max>
               <resolution>0.01</resolution>
           </range>
-          <visibility_mask>4294967294</visibility_mask>
+          <noise>
+            <type>gaussian</type>
+            <!-- Noise parameters based on published spec for Hokuyo laser
+                achieving "+-30mm" accuracy at range < 10m.  A mean of 0.0m and
+                stddev of 0.01m will put 99.7% of samples within 0.03m of the true
+                reading. -->
+            <mean>0.0</mean>
+            <stddev>0.01</stddev>
+          </noise>
+          <!-- <visibility_mask>4294967294</visibility_mask> -->
       </ray>
+    <plugin name="gazebo_ros_head_hokuyo_controller" filename="libgazebo_ros_laser.so">
+      <topicName>/scan</topicName>
+      <frameName>lidar_link</frameName>
+    </plugin>
     </sensor>
   </gazebo>

Commit message: ...

File: description/urdf/levibot.core.xacro (robot description, xacro)
@@ -156,7 +156,7 @@
     <origin xyz="0.1 0.0 0.03" rpy="0.0 0.0 0.0"/>
     <parent link="base_link"/>
-    <child link="lidar_link"/>
+    <child link="levibot/base_link/gpu_lidar"/>
   </joint>
-  <link name="lidar_link">
+  <link name="levibot/base_link/gpu_lidar">
     <collision>
       <geometry>

File: simulation/urdf/levibot.gazebo.xacro (robot description, xacro)
@@ -42,32 +42,33 @@
     </sensor>
   </gazebo> -->
-  <gazebo reference="baselink/lidar_link/gpu_lidar">
-        <sensor name='gpu_lidar' type='gpu_lidar'>
-        <pose>0 0 0 0 0 0</pose>
-          <topic>scan</topic>
-          <update_rate>10</update_rate>
-          <lidar>
-            <scan>
-              <horizontal>
-                <samples>640</samples>
-                <resolution>1</resolution>
-                <min_angle>-1.396263</min_angle>
-                <max_angle>1.396263</max_angle>
-              </horizontal>
-              <vertical>
-                <samples>1</samples>
-                <resolution>1</resolution>
-                <min_angle>0.0</min_angle>
-                <max_angle>0.0</max_angle>
-              </vertical>
-            </scan>
-            <range>
-              <min>0.08</min>
-              <max>10.0</max>
-              <resolution>0.01</resolution>
-            </range>
-          </lidar>
-          <visualize>true</visualize>
-        </sensor>
+  <gazebo reference="levibot/base_link/gpu_lidar">
+    <sensor name='gpu_lidar' type='gpu_lidar'>
+      <pose>0 0 0 0 0 0</pose>
+      <topic>scan</topic>
+      <update_rate>30</update_rate>
+      <lidar>
+        <scan>
+          <horizontal>
+            <samples>320</samples>
+            <resolution>1</resolution>
+            <min_angle>-1.396263</min_angle>
+            <max_angle>1.396263</max_angle>
+          </horizontal>
+          <vertical>
+            <samples>1</samples>
+            <resolution>1</resolution>
+            <min_angle>0.0</min_angle>
+            <max_angle>0.0</max_angle>
+          </vertical>
+        </scan>
+        <range>
+          <min>0.08</min>
+          <max>30.0</max>
+          <resolution>1</resolution>
+        </range>
+      </lidar>
+      <always_on>1</always_on>
+      <visualize>true</visualize>
+    </sensor>
   </gazebo>
 </robot>
